Commit message: Fix : Lidar Settings

File: robot_ws/configs/kros_car.xacro (robot description, xacro)
@@ -675,5 +675,5 @@
 <link name="laser"/>
   <joint name="base_to_laser" type="fixed">
-    <origin xyz="0.034 0 0.278" rpy="0 0 0"/>
+    <origin xyz="0.021 0 0.278" rpy="0 0 0"/>
     <parent link="base_link"/>
     <child link="laser"/>

Commit message: refactor: update motion arbiter control parameters, recalibrate IMU, and improve grasp approach resolution

File: robot_ws/configs/kros_car.xacro (robot description, xacro)
@@ -679,7 +679,8 @@
     <child link="laser"/>
   </joint>
+  <!--
   <link name="camera_pivot_link"/>
   <joint name="camera_pivot_joint" type="fixed">
-    <origin xyz="0.034 0 -0.04" rpy="0 0.38397 0"/> <!-- degree * 3.14159/180 -->
+    <origin xyz="0.034 0 -0.04" rpy="0 0.38397 0"/>
     <parent link="laser"/>
     <child link="camera_pivot_link"/>
@@ -691,4 +692,5 @@
     <child link="camera_link"/>
   </joint>
+  -->
   <ros2_control name="kros_car_system" type="system">
     <hardware>
